File: urack_rack/urack_rack.kicad_pcb (KiCad board)
At the start: 2 copper layers, 27 parts, among them J1 Conn_01x40, J10 Conn_01x40, J11 Conn_01x40, J12 Conn_01x40, J13 Conn_01x40, J14 Conn_01x40, J15 Conn_01x40, J16 Conn_01x40, J17 Conn_01x40, J18 Conn_01x40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

Commit message: some old changes
Parts:
- removed J10, J11, J12, J13, J14, J15, J16, J17, J18: Conn_01x40, Pin_Headers:Pin_Header_Straight_1x40_Pitch2.54mm
- removed J19, J20, J21, J22, J23, J24, J25, J26, J27: Conn_01x16, Pin_Headers:Pin_Header_Straight_1x16_Pitch2.54mm
- added REF**: MountingHole_3.2mm_M3_ISO7380, Mounting_Holes:MountingHole_3.2mm_M3_ISO7380, F.Cu at (166.1, 124.3)
- added REF**: MountingHole_3.2mm_M3_ISO7380, Mounting_Holes:MountingHole_3.2mm_M3_ISO7380, F.Cu at (159.9, 61.5)
- J1, J2, J3, J4, J5, J6, J7, J8, J9: footprint Pin_Headers:Pin_Header_Straight_1x40_Pitch2.54mm -> Pin_Headers:Pin_Header_Straight_1x40_Pitch2.54mm_SMD_Pin1Left
- moved J8 224.0 mm to (106.9, 238.8)
- moved J9 215.6 mm to (107.0, 245.7)
- moved J7 192.2 mm to (104.4, 222.2)
- moved J6 160.0 mm to (109.1, 185.9)
- moved J3 149.6 mm to (168.5, 117.2)
- moved J5 145.2 mm to (109.1, 178.9)
- moved J1 136.0 mm to (156.0, 68.6)
- moved J4 114.8 mm to (109.3, 155.5)
- moved J2 63.7 mm to (119.0, 110.3)
Other:
- board outline added: 250 x 250 mm
